Commit message: add table x table y table z joints to package syn_ur10_bringup and update model_loader module to publish respect joint state

File: syn_ur10_bringup/urdf/syn_table.urdf.xacro (robot description, xacro)
@@ -31,5 +31,5 @@
       <origin xyz="0.0 0.0 0.0" />
       <geometry>
-        <box size="5.0 5.0 0.001" />
+        <box size="8.0 8.0 0.001" />
       </geometry>
     </visual>
@@ -37,5 +37,5 @@
       <origin xyz="0.0 0.0 0.0" />
       <geometry>
-      <box size="8.0 8.0 0.001" />
+        <box size="8.0 8.0 0.001" />
       </geometry>
     </collision>
@@ -51,4 +51,7 @@
     <kd>1.0</kd>
   </gazebo>
+  <link name="table_x"/>
+  <link name="table_y"/>
+  <link name="table_z"/>
   <link name="table">
     <inertial>
@@ -111,6 +114,27 @@
     <kd>1.0</kd>
   </gazebo>
-  <joint name="floor_table_joint" type="fixed">
+  <joint name="table_floor_x_joint" type="prismatic">
     <parent link="floor"/>
+    <child link="table_x"/>
+    <origin xyz="0.0 0.0 0.0" rpy="0 0 0"/>
+    <axis xyz="1 0 0"/>
+    <limit upper="5" lower="-5" effort="1" velocity="1.00"/>
+  </joint>
+  <joint name="table_floor_y_joint" type="prismatic">
+    <parent link="table_x"/>
+    <child link="table_y"/>
+    <origin xyz="0.0 0.0 0.0" rpy="0 0 0"/>
+    <axis xyz="0 1 0"/>
+    <limit upper="5" lower="-5" effort="1" velocity="1.00"/>
+  </joint>
+  <joint name="table_floor_z_joint" type="revolute">
+    <parent link="table_y"/>
+    <child link="table_z"/>
+    <origin xyz="0.0 0.0 0.0" rpy="0 0 0"/>
+    <axis xyz="0 0 1"/>
+    <limit upper="3.1415926" lower="-3.1415926" effort="2.16" velocity="2.16"/>
+  </joint>
+  <joint name="table_z_table_joint" type="fixed">
+    <parent link="table_z"/>
     <child link="table"/>
     <origin xyz="0 0 0" rpy="0 0 0" />

File: syn_ur10_bringup/urdf/syn_ur10_setup.urdf.xacro (robot description, xacro)
@@ -7,11 +7,33 @@
   <xacro:property name="ur10_mount_height" value="0.01" />
   <link name="world" />
-  <joint name="world_floor_joint" type="fixed">
+  <joint name="floor_world_joint" type="fixed">
     <parent link="world" />
     <child link = "floor" />
     <origin xyz="0.0 0.0 0.0" rpy="0.0 0.0 0.0" />
   </joint>
+  <!-- <link name="aircraft_frame">
+    <inertial>
+      <mass value="20000" />
+      <origin xyz="0 0 0" />
+      <inertia  ixx="0.01" ixy="0" ixz="0" iyy="0.01" iyz="0" izz="0.01" />
+    </inertial>
+    <visual>
+      <geometry>
+        <mesh filename="package://syn_ur10_bringup/meshes/M1-2-010-0-001-A_Jig-Aussenhaut-FAL.stl" scale="0.001 0.001 0.001" />
+      </geometry>
+    </visual>
+    <collision>
+      <geometry>
+        <mesh filename="package://syn_ur10_bringup/meshes/M1-2-010-0-001-A_Jig-Aussenhaut-FAL.stl" scale="0.001 0.001 0.001" />
+      </geometry>
+    </collision>
+  </link>
+  <joint name="aircraft_frame_world_joint" type="fixed">
+    <parent link="world"/>
+    <child link="aircraft_frame" />
+    <origin xyz="0.0 0.0 0.53" rpy="0.0 0.0 0.0" />
+  </joint> -->
   <link name="map" />
-  <joint name="map_world" type="fixed">
+  <joint name="map_world_joint" type="fixed">
     <parent link="world" />
     <child link = "map" />

Commit message: modify module [syn_ur10_bringup]: add urdf file for tools, update table urdf file to make table movable, update SRDF file for new robot configuration

File: syn_ur10_bringup/urdf/syn_table.urdf.xacro (robot description, xacro)
@@ -3,13 +3,11 @@
   <xacro:arg name="floating_table" default="false" />
   <xacro:property name="roomheight" value="3.0" />
-  <xacro:property name="tableheight" value="0.86" />
-  <xacro:property name="tablewidth" value="0.61" />
+  <xacro:property name="tableheight" value="0.83" />
+  <xacro:property name="tablewidth" value="0.83" />
   <xacro:property name="tabledepth" value="0.9" />
-  <xacro:property name="ur10_mount_height" value="0.01" />
-  <xacro:property name="ur10_mount_width" value="0.2" />
-  <xacro:property name="ur10_mount_depth" value="0.2" />
+  <xacro:property name="ur10_mount_offset_y" value="-0.212" />
   <xacro:property name="scan_offset_x" value="0.00" />
-  <xacro:property name="scan_offset_y" value="-0.32" />
-  <xacro:property name="scan_offset_z" value="0.03" />
+  <xacro:property name="scan_offset_y" value="-0.40" />
+  <xacro:property name="scan_offset_z" value="0.095" />
   <material name="white">
     <color rgba="1 1 1 1"/>
@@ -51,7 +49,4 @@
     <kd>1.0</kd>
   </gazebo>
-  <link name="table_x"/>
-  <link name="table_y"/>
-  <link name="table_z"/>
   <link name="table">
     <inertial>
@@ -84,64 +79,10 @@
   </gazebo>
   <link name="table_top"/>
+  <link name="ur10_mount"/>
   <link name="scan"/>
-  <link name="ur10_mount">
-    <inertial>
-      <origin xyz="0 0 ${ur10_mount_height/2}" />
-      <mass value="2000" />
-      <inertia  ixx="1" ixy="0" ixz="0" iyy="1" iyz="0" izz="1" />
-    </inertial>
-    <visual>
-      <material name="lightgray" />
-      <origin xyz="0.0 0.0 ${ur10_mount_height/2}" />
-      <geometry>
-        <box size="${ur10_mount_width} ${ur10_mount_depth} ${ur10_mount_height}" />
-      </geometry>
-    </visual>
-    <collision>
-      <origin xyz="0.0 0.0 ${ur10_mount_height/2}" />
-      <geometry>
-        <box size="${ur10_mount_width} ${ur10_mount_depth} ${ur10_mount_height}" />
-      </geometry>
-    </collision>
-  </link>
-  <gazebo reference="ur10_mount">
-    <material>Gazebo/Blue</material>
-    <turnGravityOff>false</turnGravityOff>
-    <selfCollide>true</selfCollide>
-    <mu1>100.0</mu1>
-    <mu2>100.0</mu2>
-    <kp>1000000.0</kp>
-    <kd>1.0</kd>
-  </gazebo>
-  <joint name="table_floor_x_joint" type="prismatic">
+  <joint name="table_floor_joint" type="floating">
     <parent link="floor"/>
-    <child link="table_x"/>
-    <origin xyz="0.0 0.0 0.0" rpy="0 0 0"/>
-    <axis xyz="1 0 0"/>
-    <limit upper="5" lower="-5" effort="1" velocity="1.00"/>
-  </joint>
-  <joint name="table_floor_y_joint" type="prismatic">
-    <parent link="table_x"/>
-    <child link="table_y"/>
-    <origin xyz="0.0 0.0 0.0" rpy="0 0 0"/>
-    <axis xyz="0 1 0"/>
-    <limit upper="5" lower="-5" effort="1" velocity="1.00"/>
-  </joint>
-  <joint name="table_floor_z_joint" type="revolute">
-    <parent link="table_y"/>
-    <child link="table_z"/>
-    <origin xyz="0.0 0.0 0.0" rpy="0 0 0"/>
-    <axis xyz="0 0 1"/>
-    <limit upper="3.1415926" lower="-3.1415926" effort="2.16" velocity="2.16"/>
-  </joint>
-  <joint name="table_z_table_joint" type="fixed">
-    <parent link="table_z"/>
     <child link="table"/>
     <origin xyz="0 0 0" rpy="0 0 0" />
-  </joint>
-  <joint name="table_mount_joint" type="fixed">
-    <parent link="table"/>
-    <child link="ur10_mount"/>
-	  <origin xyz="0 -0.16 ${tableheight}" rpy="0 0 0" />
   </joint>
   <joint name="table_top_joint" type="fixed">
@@ -150,6 +91,11 @@
 	  <origin xyz="0 0 ${tableheight}" rpy="0 0 0" />
   </joint>
-  <joint name="mount_scan_joint" type="fixed">
-    <parent link="ur10_mount"/>
+  <joint name="ur10_mount_table_top_joint" type="fixed">
+    <parent link="table_top"/>
+    <child link="ur10_mount"/>
+	  <origin xyz="0 ${ur10_mount_offset_y} 0" rpy="0 0 0" />
+  </joint>
+  <joint name="scan_table_top_joint" type="fixed">
+    <parent link="table_top"/>
     <child link="scan"/>
 	  <origin xyz="${scan_offset_x} ${scan_offset_y} ${scan_offset_z}" rpy="0 0 0" />

File: syn_ur10_bringup/urdf/syn_ur10_setup.urdf.xacro (robot description, xacro)
@@ -5,4 +5,6 @@
   <!-- arm -->
   <xacro:include filename="$(find syn_ur10_bringup)/urdf/arm.urdf.xacro" />
+  <!-- tool -->
+  <xacro:include filename="$(find syn_ur10_bringup)/urdf/tool.urdf.xacro" />
   <xacro:property name="ur10_mount_height" value="0.01" />
   <link name="world" />
@@ -12,26 +14,4 @@
     <origin xyz="0.0 0.0 0.0" rpy="0.0 0.0 0.0" />
   </joint>
-  <!-- <link name="aircraft_frame">
-    <inertial>
-      <mass value="20000" />
-      <origin xyz="0 0 0" />
-      <inertia  ixx="0.01" ixy="0" ixz="0" iyy="0.01" iyz="0" izz="0.01" />
-    </inertial>
-    <visual>
-      <geometry>
-        <mesh filename="package://syn_ur10_bringup/meshes/M1-2-010-0-001-A_Jig-Aussenhaut-FAL.stl" scale="0.001 0.001 0.001" />
-      </geometry>
-    </visual>
-    <collision>
-      <geometry>
-        <mesh filename="package://syn_ur10_bringup/meshes/M1-2-010-0-001-A_Jig-Aussenhaut-FAL.stl" scale="0.001 0.001 0.001" />
-      </geometry>
-    </collision>
-  </link>
-  <joint name="aircraft_frame_world_joint" type="fixed">
-    <parent link="world"/>
-    <child link="aircraft_frame" />
-    <origin xyz="0.0 0.0 0.53" rpy="0.0 0.0 0.0" />
-  </joint> -->
   <link name="map" />
   <joint name="map_world_joint" type="fixed">
@@ -43,5 +23,10 @@
     <parent link="ur10_mount" />
     <child link = "ur10_base_link" />
-    <origin xyz="0.0 0.0 ${ur10_mount_height}" rpy="0.0 0.0 0.0" />
+    <origin xyz="0.0 0.0 ${ur10_mount_height}" rpy="0.0 0.0 ${radians(90)}" />
+  </joint>
+  <joint name="ur10_tool_joint" type="fixed">
+    <parent link="ur10_tool0" />
+    <child link = "tool_base" />
+    <origin xyz="0.0 0.0 0.0" rpy="0.0 0.0 0.0" />
   </joint>
 </robot>

Commit message: rename module 'opencv_test' to 'object_localizer'; update syn_ur10 urdf file and moveit configuration; update 'model_loader' module to handle unstable scan readings

File: syn_ur10_bringup/urdf/syn_table.urdf.xacro (robot description, xacro)
@@ -9,5 +9,5 @@
   <xacro:property name="scan_offset_x" value="0.00" />
   <xacro:property name="scan_offset_y" value="-0.40" />
-  <xacro:property name="scan_offset_z" value="0.095" />
+  <xacro:property name="scan_offset_z" value="0.06" />
   <material name="white">
     <color rgba="1 1 1 1"/>
@@ -80,5 +80,24 @@
   <link name="table_top"/>
   <link name="ur10_mount"/>
-  <link name="scan"/>
+  <link name="scan">
+    <inertial>
+      <origin xyz="0.0 0.0 0.0" />
+      <mass value="200" />
+      <inertia  ixx="1" ixy="0" ixz="0" iyy="1" iyz="0" izz="1" />
+    </inertial>
+    <visual>
+      <material name="lightgray" />
+      <origin xyz="0.0 0.0 0.0" />
+      <geometry>
+        <box size="0.10 0.10 0.12" />
+      </geometry>
+    </visual>
+    <collision>
+      <origin xyz="0.0 0.0 0.0" />
+      <geometry>
+        <box size="0.10 0.10 0.12" />
+      </geometry>
+    </collision>
+  </link>
   <joint name="table_floor_joint" type="floating">
     <parent link="floor"/>
