Commit message: add node [rivet_localizer] and [point_rivet]

File: syn_ur10_bringup/urdf/tool.urdf.xacro (robot description, xacro)
@@ -2,4 +2,12 @@
 <robot xmlns:xacro="http://www.ros.org/wiki/xacro" name="tool" >
   <xacro:include filename="$(find microepsilon_scancontrol)/description/urdf/scanCONTROL_2900-50_macro.urdf.xacro" />
+  <xacro:property name="rivet_tool_part_1_length" value="0.07415" />
+  <xacro:property name="rivet_tool_part_1_radius" value="0.015" />
+  <xacro:property name="rivet_tool_part_2_height" value="0.012" />
+  <xacro:property name="rivet_tool_part_2_length" value="0.0625" />
+  <xacro:property name="rivet_tool_part_2_width" value="0.03" />
+  <xacro:property name="rivet_tool_part_3_length" value="0.044" />
+  <xacro:property name="rivet_tool_part_3_radius" value="0.0075" />
+  <xacro:property name="rivet_tool_offset" value="0.000" />
   <link name="tool_base">
     <inertial>
@@ -22,4 +30,87 @@
     </collision>
   </link>
+  <link name="rivet_tool_part_1">
+    <inertial>
+      <origin xyz="0.0 0.0 0.0" />
+      <mass value="200" />
+      <inertia  ixx="1" ixy="0" ixz="0" iyy="1" iyz="0" izz="1" />
+    </inertial>
+    <visual>
+      <material name="black" />
+      <origin xyz="0.0 0.0 ${rivet_tool_part_1_length/2}" />
+      <geometry>
+        <cylinder radius="${rivet_tool_part_1_radius}" length="${rivet_tool_part_1_length}" />
+      </geometry>
+    </visual>
+    <collision>
+      <origin xyz="0.0 0.0 ${rivet_tool_part_1_length/2}" />
+      <geometry>
+        <cylinder radius="${rivet_tool_part_1_radius}" length="${rivet_tool_part_1_length}" />
+      </geometry>
+    </collision>
+  </link>
+  <!--change this property to offset the -->
+  <xacro:property name="rivet_tool_part_1_z_offset" value="0.0006" />
+  <joint name="tool_base_rivet_tool_part_1_joint" type="fixed">
+    <parent link="tool_base"/>
+    <child link="rivet_tool_part_1"/>
+    <origin xyz="0 -0.03275 ${0.03787 + rivet_tool_part_1_z_offset}" rpy="${radians(90)} 0 0" />
+  </joint>
+  <link name="rivet_tool_part_2">
+    <inertial>
+      <origin xyz="0.0 0.0 0.0" />
+      <mass value="200" />
+      <inertia  ixx="1" ixy="0" ixz="0" iyy="1" iyz="0" izz="1" />
+    </inertial>
+    <visual>
+      <material name="black" />
+      <origin xyz="0.0 0.0 0.0" />
+      <geometry>
+        <box size="${rivet_tool_part_2_length} ${rivet_tool_part_2_width} ${rivet_tool_part_2_height}" />
+      </geometry>
+    </visual>
+    <collision>
+      <origin xyz="0.0 0.0 0.0" />
+      <geometry>
+        <box size="${rivet_tool_part_2_length} ${rivet_tool_part_2_width} ${rivet_tool_part_2_height}" />
+      </geometry>
+    </collision>
+  </link>
+  <joint name="rivet_tool_part_1_rivet_tool_part_2_joint" type="fixed">
+    <parent link="rivet_tool_part_1"/>
+    <child link="rivet_tool_part_2"/>
+    <origin xyz="${-rivet_tool_part_2_length/2} 0 ${rivet_tool_part_1_length + rivet_tool_part_2_height/2}" rpy="0 0 0" />
+  </joint>
+  <link name="rivet_tool_part_3">
+    <inertial>
+      <origin xyz="0.0 0.0 0.0" />
+      <mass value="200" />
+      <inertia  ixx="1" ixy="0" ixz="0" iyy="1" iyz="0" izz="1" />
+    </inertial>
+    <visual>
+      <material name="black" />
+      <origin xyz="0.0 0.0 ${rivet_tool_part_3_length/2}" />
+      <geometry>
+        <cylinder radius="${rivet_tool_part_3_radius}" length="${rivet_tool_part_3_length}" />
+      </geometry>
+    </visual>
+    <collision>
+      <origin xyz="0.0 0.0 ${rivet_tool_part_3_length/2}" />
+      <geometry>
+        <cylinder radius="${rivet_tool_part_3_radius}" length="${rivet_tool_part_3_length}" />
+      </geometry>
+    </collision>
+  </link>
+  <joint name="rivet_tool_part_2_rivet_tool_part_3_joint" type="fixed">
+    <parent link="rivet_tool_part_2"/>
+    <child link="rivet_tool_part_3"/>
+    <origin xyz="${-rivet_tool_part_2_length/2} 0 ${rivet_tool_part_2_height/2}" rpy="${radians(0)} 0 0" />
+  </joint>
+  <link name="rivet_tool" />
+  <joint name="rivet_tool_part_3_rivet_tool_joint" type="fixed">
+    <parent link="rivet_tool_part_3"/>
+    <child link="rivet_tool"/>
+    <origin xyz="0 0 ${rivet_tool_part_3_length + rivet_tool_offset}" rpy="${radians(-90)} ${radians(90)} 0" />
+  </joint>
   <!-- scanCONTROL_2900-50  sensor -->
   <xacro:scanCONTROL_2900-50 prefix="scanCONTROL_2900-50_" parent="tool_base">

Commit message: add parameters [rivet_tool_x[y][z]_offset] to adjust the offset the tool frame

File: syn_ur10_bringup/urdf/tool.urdf.xacro (robot description, xacro)
@@ -1,13 +1,18 @@
 <?xml version="1.0"?>
 <robot xmlns:xacro="http://www.ros.org/wiki/xacro" name="tool" >
+  <!-- change the value of rivet_tool_x_offset to adjust x offset -->
+  <xacro:property name="rivet_tool_x_offset" value="0.050" />
+  <!-- change the value of rivet_tool_y_adjust to adjust y offset -->
+  <xacro:property name="rivet_tool_y_adjust" value="0.0000" />
+  <!-- change the value of rivet_tool_z_adjust to adjust z offset -->
+  <xacro:property name="rivet_tool_z_adjust" value="0.0006" />
   <xacro:include filename="$(find microepsilon_scancontrol)/description/urdf/scanCONTROL_2900-50_macro.urdf.xacro" />
   <xacro:property name="rivet_tool_part_1_length" value="0.07415" />
   <xacro:property name="rivet_tool_part_1_radius" value="0.015" />
   <xacro:property name="rivet_tool_part_2_height" value="0.012" />
-  <xacro:property name="rivet_tool_part_2_length" value="0.0625" />
+  <xacro:property name="rivet_tool_part_2_length" value="${0.0625 - rivet_tool_y_adjust}" />
   <xacro:property name="rivet_tool_part_2_width" value="0.03" />
   <xacro:property name="rivet_tool_part_3_length" value="0.044" />
   <xacro:property name="rivet_tool_part_3_radius" value="0.0075" />
-  <xacro:property name="rivet_tool_offset" value="0.000" />
   <link name="tool_base">
     <inertial>
@@ -50,10 +55,8 @@
     </collision>
   </link>
-  <!--change this property to offset the -->
-  <xacro:property name="rivet_tool_part_1_z_offset" value="0.0006" />
   <joint name="tool_base_rivet_tool_part_1_joint" type="fixed">
     <parent link="tool_base"/>
     <child link="rivet_tool_part_1"/>
-    <origin xyz="0 -0.03275 ${0.03787 + rivet_tool_part_1_z_offset}" rpy="${radians(90)} 0 0" />
+    <origin xyz="0 -0.03275 ${0.03787 + rivet_tool_y_adjust}" rpy="${radians(90)} 0 0" />
   </joint>
   <link name="rivet_tool_part_2">
@@ -111,5 +114,5 @@
     <parent link="rivet_tool_part_3"/>
     <child link="rivet_tool"/>
-    <origin xyz="0 0 ${rivet_tool_part_3_length + rivet_tool_offset}" rpy="${radians(-90)} ${radians(90)} 0" />
+    <origin xyz="0 0 ${rivet_tool_part_3_length + rivet_tool_x_offset}" rpy="${radians(-90)} ${radians(90)} 0" />
   </joint>
   <!-- scanCONTROL_2900-50  sensor -->

Commit message: adjust the xyz position of rivet tool frame

File: syn_ur10_bringup/urdf/tool.urdf.xacro (robot description, xacro)
@@ -2,11 +2,11 @@
 <robot xmlns:xacro="http://www.ros.org/wiki/xacro" name="tool" >
   <!-- change the value of rivet_tool_x_offset to adjust x offset -->
-  <xacro:property name="rivet_tool_x_offset" value="0.050" />
+  <xacro:property name="rivet_tool_x_offset" value="0.000" />
   <!-- change the value of rivet_tool_y_adjust to adjust y offset -->
-  <xacro:property name="rivet_tool_y_adjust" value="0.0000" />
+  <xacro:property name="rivet_tool_y_adjust" value="0.005" />
   <!-- change the value of rivet_tool_z_adjust to adjust z offset -->
-  <xacro:property name="rivet_tool_z_adjust" value="0.0006" />
+  <xacro:property name="rivet_tool_z_adjust" value="0.0005" />
   <xacro:include filename="$(find microepsilon_scancontrol)/description/urdf/scanCONTROL_2900-50_macro.urdf.xacro" />
-  <xacro:property name="rivet_tool_part_1_length" value="0.07415" />
+  <xacro:property name="rivet_tool_part_1_length" value="0.07015" />
   <xacro:property name="rivet_tool_part_1_radius" value="0.015" />
   <xacro:property name="rivet_tool_part_2_height" value="0.012" />
@@ -58,5 +58,5 @@
     <parent link="tool_base"/>
     <child link="rivet_tool_part_1"/>
-    <origin xyz="0 -0.03275 ${0.03787 + rivet_tool_y_adjust}" rpy="${radians(90)} 0 0" />
+    <origin xyz="0 -0.03275 ${0.03787 + rivet_tool_z_adjust}" rpy="${radians(90)} 0 0" />
   </joint>
   <link name="rivet_tool_part_2">

Commit message: change the z axis offset in urdf file; change the generate the point rivet path in node [rivet_localizer]

File: syn_ur10_bringup/urdf/tool.urdf.xacro (robot description, xacro)
@@ -6,5 +6,5 @@
   <xacro:property name="rivet_tool_y_adjust" value="0.005" />
   <!-- change the value of rivet_tool_z_adjust to adjust z offset -->
-  <xacro:property name="rivet_tool_z_adjust" value="0.0005" />
+  <xacro:property name="rivet_tool_z_adjust" value="0.000" />
   <xacro:include filename="$(find microepsilon_scancontrol)/description/urdf/scanCONTROL_2900-50_macro.urdf.xacro" />
   <xacro:property name="rivet_tool_part_1_length" value="0.07015" />

Commit message: adjust the rivet tool along the y axiz for +0.5mm

File: syn_ur10_bringup/urdf/tool.urdf.xacro (robot description, xacro)
@@ -4,5 +4,5 @@
   <xacro:property name="rivet_tool_x_offset" value="0.000" />
   <!-- change the value of rivet_tool_y_adjust to adjust y offset -->
-  <xacro:property name="rivet_tool_y_adjust" value="0.005" />
+  <xacro:property name="rivet_tool_y_adjust" value="0.0055" />
   <!-- change the value of rivet_tool_z_adjust to adjust z offset -->
   <xacro:property name="rivet_tool_z_adjust" value="0.000" />

Commit message: update the urdf model of tool, define new poses, using tf_dummny to fix the table to the floor, and update the rviz content

File: syn_ur10_bringup/urdf/tool.urdf.xacro (robot description, xacro)
@@ -83,5 +83,5 @@
     <parent link="rivet_tool_part_1"/>
     <child link="rivet_tool_part_2"/>
-    <origin xyz="${-rivet_tool_part_2_length/2} 0 ${rivet_tool_part_1_length + rivet_tool_part_2_height/2}" rpy="0 0 0" />
+    <origin xyz="0 ${rivet_tool_part_2_length/2} ${rivet_tool_part_1_length + rivet_tool_part_2_height/2}" rpy="0 0 ${radians(-90)}" />
   </joint>
   <link name="rivet_tool_part_3">
@@ -116,8 +116,5 @@
     <origin xyz="0 0 ${rivet_tool_part_3_length + rivet_tool_x_offset}" rpy="${radians(-90)} ${radians(90)} 0" />
   </joint>
-  <!-- scanCONTROL_2900-50  sensor -->
-  <xacro:scanCONTROL_2900-50 prefix="scanCONTROL_2900-50_" parent="tool_base">
-    <origin xyz="0.0617 -0.09003 0.0870" rpy="${radians(0)} ${radians(0)} ${radians(0)}" />
-  </xacro:scanCONTROL_2900-50>
+  <!-- link camera_plate and link to tool_base -->
   <link name="camera_plate">
     <inertial>
@@ -128,5 +125,5 @@
     <visual>
       <material name="lightgray" />
-      <origin xyz="0.0392 -0.0298 0.076" />
+      <origin xyz="0.0 0.0 0.0" />
       <geometry>
         <box size="0.003 0.126 0.132" />
@@ -134,5 +131,5 @@
     </visual>
     <collision>
-      <origin xyz="0.0392 -0.0298 0.076" />
+      <origin xyz="0.0 0.0 0.0" />
       <geometry>
         <box size="0.003 0.126 0.132" />
@@ -143,6 +140,11 @@
     <parent link="tool_base"/>
     <child link="camera_plate"/>
-    <origin xyz="0 0 0" rpy="0 0 0" />
+    <origin xyz="-0.0392 0.0298 0.069" rpy="0 0 0" />
   </joint>
+  <!-- scanCONTROL_2900-50 sensor and is connected to tool_base frame -->
+  <xacro:scanCONTROL_2900-50 prefix="scanCONTROL_2900-50_" parent="tool_base">
+    <origin xyz="-0.060 0.09 0.078" rpy="${radians(0)} ${radians(0)} ${radians(180)}" />
+  </xacro:scanCONTROL_2900-50>
+  <!-- camera_support link is connected to scanCONTROL_2900-50_scanner_link -->
   <link name="camera_support">
     <inertial>
@@ -168,5 +170,5 @@
     <parent link="scanCONTROL_2900-50_scanner_link"/>
     <child link="camera_support"/>
-    <origin xyz="0 0.0085 0.032" rpy="0.0 ${radians(90)} 0.0" />
+    <origin xyz="0 0.09 0.045" rpy="0.0 ${radians(90)} 0.0" />
   </joint>
   <link name="camera_support_2" />
@@ -176,4 +178,5 @@
     <origin xyz="0 0.0 0.0208" rpy="0.0 ${radians(0)} ${radians(180)}" />
   </joint>
+  <!-- connect camera to link camera_support_2 -->
   <xacro:include filename="$(find realsense2_camera)/urdf/_r430.urdf.xacro"/>
   <sensor_r430 parent="camera_support_2">

Commit message: adjust the position of rivet_tool frame (by adding new parameters: rivet_tool_distance_offsetrivet_tool_horizontal_adjust, rivet_tool_vertical_adjust)

File: syn_ur10_bringup/urdf/tool.urdf.xacro (robot description, xacro)
@@ -1,18 +1,19 @@
 <?xml version="1.0"?>
-<robot xmlns:xacro="http://www.ros.org/wiki/xacro" name="tool" >
-  <!-- change the value of rivet_tool_x_offset to adjust x offset -->
-  <xacro:property name="rivet_tool_x_offset" value="0.000" />
-  <!-- change the value of rivet_tool_y_adjust to adjust y offset -->
-  <xacro:property name="rivet_tool_y_adjust" value="0.0055" />
-  <!-- change the value of rivet_tool_z_adjust to adjust z offset -->
-  <xacro:property name="rivet_tool_z_adjust" value="0.000" />
+<robot xmlns:xacro="http://www.ros.org/wiki/xacro" name="tool">
+  <!-- change the value of rivet_tool_distance_offset to adjust the distance to the target-->
+  <xacro:property name="rivet_tool_distance_offset" value="0.0000" />
+  <!-- change the value of rivet_tool_horizontal_adjust to adjust the tool horizontally, plus for left and minus for right -->
+  <xacro:property name="rivet_tool_horizontal_adjust" value="-0.0047" />
+  <!-- change the value of rivet_tool_vertical_adjust to adjust the tool vertically, plus for up and minus for down -->
+  <xacro:property name="rivet_tool_vertical_adjust" value="-0.0015" />
   <xacro:include filename="$(find microepsilon_scancontrol)/description/urdf/scanCONTROL_2900-50_macro.urdf.xacro" />
-  <xacro:property name="rivet_tool_part_1_length" value="0.07015" />
+  <xacro:property name="rivet_tool_part_1_length" value="0.05078" />
   <xacro:property name="rivet_tool_part_1_radius" value="0.015" />
   <xacro:property name="rivet_tool_part_2_height" value="0.012" />
-  <xacro:property name="rivet_tool_part_2_length" value="${0.0625 - rivet_tool_y_adjust}" />
+  <xacro:property name="rivet_tool_part_2_length" value="0.066" />
   <xacro:property name="rivet_tool_part_2_width" value="0.03" />
-  <xacro:property name="rivet_tool_part_3_length" value="0.044" />
+  <xacro:property name="rivet_tool_part_3_length" value="0.06374" />
   <xacro:property name="rivet_tool_part_3_radius" value="0.0075" />
+  <xacro:property name="rivet_tool_angle" value="154.6" />
   <link name="tool_base">
     <inertial>
@@ -58,5 +59,6 @@
     <parent link="tool_base"/>
     <child link="rivet_tool_part_1"/>
-    <origin xyz="0 -0.03275 ${0.03787 + rivet_tool_z_adjust}" rpy="${radians(90)} 0 0" />
+    <!-- <origin xyz="0 -0.03275 ${0.03787 + rivet_tool_z_adjust}" rpy="${radians(90)} 0 0" /> -->
+    <origin xyz="${0 - rivet_tool_horizontal_adjust} -0.03275 ${0.03787 - rivet_tool_vertical_adjust}" rpy="${radians(90)} ${radians(rivet_tool_angle)} 0" />
   </joint>
   <link name="rivet_tool_part_2">
@@ -114,5 +116,5 @@
     <parent link="rivet_tool_part_3"/>
     <child link="rivet_tool"/>
-    <origin xyz="0 0 ${rivet_tool_part_3_length + rivet_tool_x_offset}" rpy="${radians(-90)} ${radians(90)} 0" />
+    <origin xyz="0 0 ${rivet_tool_part_3_length + rivet_tool_distance_offset}" rpy="${radians(-90)} ${radians(90)} ${radians(90+rivet_tool_angle)}" />
   </joint>
   <!-- link camera_plate and link to tool_base -->
